File: KRYZBO HE.kicad_sch (KiCad schematic)
At the start: 44 parts, among them SW1 SW_SPST, SW2 SW_DIP_x04, U1 AMS1117-3.3, U2 74LS08, U3 STM32F303CBTx, U5 H5VU25U, Y1 16MHz

Commit message: Add files via upload
Parts:
- removed BZ1: AST1109MLTRQ, MoonBoard:AST1109MLTRQ, symbol Device:Buzzer
- removed C1, C2: 2u2, Capacitor_SMD:C_0805_2012Metric, symbol Device:C_Small
- removed FB1: 120R @ 100MHz, Inductor_SMD:L_0805_2012Metric, symbol Device:FerriteBead_Small
- removed SW2: SW_DIP_x04, Button_Switch_THT:SW_DIP_SPSTx04_Slide_6.7x11.72mm_W7.62mm_P2.54mm_LowProfile, symbol Switch:SW_DIP_x04
- removed SWD1: Conn_02x03_Odd_Even, Connector_PinHeader_2.54mm:PinHeader_2x03_P2.54mm_Vertical, symbol Connector_Generic:Conn_02x03_Odd_Even
- removed TH1, TH2, TH3: ToolingHole, MoonBoard:JLC-Tooling-Hole, symbol Mechanical:MountingHole
- removed U2: 74LS08, Package_SO:SOIC-14_3.9x8.7mm_P1.27mm, symbol 74xx:74LS08
- removed U5 (x2): H5VU25U, MoonBoard:DFN2510, symbol Unified-Daughterboard-rescue:TPD4E05U06DQAR-acheronSymbols
- removed USB1: X1224WRS-04-LPV01, MoonBoard:PicoEZMate-Reinforced-Alt, symbol Connector_Generic_MountingPin:Conn_01x04_MountingPin
- added D7: PRTR5V0U2X, Package_TO_SOT_SMD:SOT-143, symbol Power_Protection:PRTR5V0U2X
- added F1: 1.1A, Fuse:Fuse_1206_3216Metric, symbol Device:Polyfuse
- added J3: USB-C 2.0 Receptacle, Connector_USB:USB_C_Receptacle_HRO_TYPE-C-31-M-12, symbol Connector:USB_C_Receptacle_USB2.0
- added R2, R6: 5.1k, Resistor_SMD:R_0402_1005Metric, symbol Device:R
Connections:
- net +5V: now also D7.4 (VCC), F1.2
- net GND: now also D7.1 (GND), J3.A1 (GND), J3.A12 (GND), J3.B1 (GND), J3.B12 (GND), J3.S1 (SHIELD), R2.1, R6.1
- net USB_D+: now also D7.2 (I/O1), J3.A6 (D+), J3.B6 (D+)
- net USB_D-: now also D7.3 (I/O2), J3.A7 (D-), J3.B7 (D-)
- net VBUS: now also F1.1, J3.A4 (VBUS), J3.A9 (VBUS), J3.B4 (VBUS), J3.B9 (VBUS)
- net DAC1_OUT1: no longer names the net of U3.14 (PA4)
- net DAC1_OUT2: no longer names the net of U3.15 (PA5)
- net ENCODER_A: no longer names the net of U3.10 (PA0)
- net ENCODER_B: no longer names the net of U3.11 (PA1)
- new net: J3.B5 (CC2), R6.2
- new net: J3.A5 (CC1), R2.2
- no-connect marks 17 -> 14
Other:
- note added: "Power"
- note removed: "DIP Selector Switch"
- note removed: "JLCPCB Tooling"
- note removed: "OLED"
- note removed: "SWD Connector"
- note removed: "Unused AND Gates"
- note removed: "uDB Connector"
