File: keys.kicad_sch (KiCad schematic)
At the start: 0 parts

Commit message: Add files via upload
Other:
- removed sheet sensor13
- removed sheet sensor14
- removed sheet sensor15
- removed sheet sensor16
- removed sheet sensor47
- removed sheet sensor48
- removed sheet sensor75
- removed sheet sensor80
